File: Project_PCB_Subsystem/Project_PCB_Subsystem.kicad_pcb (KiCad board)
At the start: 2 copper layers, 10 parts, among them U1 ESP32-C6 Microcontroller

Commit message: Updated PCB design file folder
Routing:
- net GND: track 0.00 -> 286.1 mm, vias 0 -> 2
- net VCC: track 0.00 -> 205.1 mm, vias 0 -> 3
- net Net-(KS1-Pin_1): track 0.00 -> 64.4 mm, vias 0 -> 1
- net Net-(KS1-Pin_2): track 0.00 -> 58.6 mm, vias 0 -> 1
- net Net-(B1-B): track 0.00 -> 57.3 mm
- net Net-(LS1-Pin_3): track 0.00 -> 54.3 mm, vias 0 -> 3
- net Net-(KS1-Pin_3): track 0.00 -> 52.8 mm, vias 0 -> 1
- net Net-(LS1-Pin_4): track 0.00 -> 51.3 mm, vias 0 -> 3
- net Net-(KS1-Pin_4): track 0.00 -> 45.2 mm, vias 0 -> 1
- net Net-(U1-IO9): track 0.00 -> 45.0 mm, vias 0 -> 1
- net Net-(RV1-Pad1): track 0.00 -> 43.6 mm, vias 0 -> 1
- net Net-(U1-IO8): track 0.00 -> 40.7 mm, vias 0 -> 1
- net Net-(KS1-Pin_5): track 0.00 -> 38.8 mm, vias 0 -> 1
- net Net-(KS1-Pin_6): track 0.00 -> 34.1 mm, vias 0 -> 1
- net Net-(KS1-Pin_7): track 0.00 -> 28.4 mm, vias 0 -> 1
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Other:
- board outline added: 89 x 123.5 mm
